File: hardware/valdiklis/valdiklis.sch (KiCad schematic (older format))
At the start: 5 parts, among them M1 unicon_v1, U1 DHT11, U2 L298HN, U3 DHT11

Commit message: pcb plokstes ir schemos paruosimas
Parts:
- added C1, C13, C14, C2, C3, C4, C5, C6, C7, C8, C9: 0.1, Capacitor_SMD:C_1206_3216Metric, symbol Device:C
- added C10: CP, Capacitor_THT:CP_Radial_D5.0mm_P2.50mm, symbol Device:CP
- added C11, C12: CP, Capacitor_THT:CP_Radial_D10.0mm_P5.00mm, symbol Device:CP
- added D1: D, Diode_SMD:D_MELF, symbol Device:D
- added D2: D, Diode_THT:D_DO-27_P15.24mm_Horizontal, symbol Device:D
- added J1: POWER, Connector_Phoenix_MSTB:PhoenixContact_MSTBA_2,5_4-G-5,08_1x04_P5.08mm_Horizontal, symbol Connector_Generic:Conn_01x04
- added J2: UART, Connector_PinHeader_2.54mm:PinHeader_1x03_P2.54mm_Vertical, symbol Connector_Generic:Conn_01x03
- added R10, R11: 4,7k, Resistor_SMD:R_0805_2012Metric, symbol Device:R
- added R2, R3, R4, R5, R6: 10k, Resistor_SMD:R_0805_2012Metric, symbol Device:R
- added R7: 1R0, Resistor_THT:R_Axial_DIN0207_L6.3mm_D2.5mm_P10.16mm_Horizontal, symbol Device:R
- added R8, R9: 47R, Resistor_SMD:R_0805_2012Metric, symbol Device:R
- added RV1, RV2: 5k, Potentiometer_THT:Potentiometer_Piher_PT-6-V_Vertical, symbol Device:R_POT_TRIM
- added SW1, SW2: RESET, Button_Switch_THT:SW_PUSH_6mm_H5mm, symbol mech:SW_TACT_6301
- M1: value unicon_v1 -> UniCon; symbol unicon:unicon_v1 -> valdiklis-rescue:unicon_v1-unicon
- R1: value R -> 1R0; footprint (none) -> Resistor_THT:R_Axial_DIN0207_L6.3mm_D2.5mm_P10.16mm_Horizontal
- U1, U3: symbol dht11:DHT11 -> valdiklis-rescue:DHT11-dht11
Connections:
- net labels added: 12V1, 3VDC, AD1, AD2, ADC, BOOT, GND1, L298_ENA, L298_IN1, L298_IN2, UART_RX, UART_TX, ~RST
- net labels removed: ENA, IN1, IN2
- wire segments 42 -> 149
Other:
- moved on the sheet: R1, U2

Commit message: pcb ir schemos paruosimas
Parts:
- added D3, D4, D5, D6: D, Diode_SMD:D_SMA, symbol Device:D
- added R12, R13: 4,7k, Resistor_SMD:R_0805_2012Metric, symbol Device:R
- C5, C6: footprint Capacitor_SMD:C_1206_3216Metric -> Capacitor_SMD:C_0805_2012Metric
- C7, C9: value 0.1 -> 1.0
- SW1, SW2: symbol mech:SW_TACT_6301 -> valdiklis-rescue:SW_TACT_6301-mech
Connections:
- wire segments 149 -> 168
Other:
- moved on the sheet: C1, C4, C5, C6, C7, R10, R11, R8, R9, U1, U3
