File: hardware/valdiklis/valdiklis.kicad_pcb (KiCad board)
At the start: 2 copper layers, 59 x 67 mm, 4 parts, among them M1 unicon_v1, U1 DHT11, U2 L298HN, U3 DHT11

Commit message: pcb plokstes ir schemos paruosimas
Parts:
- added C1: 0.1, Capacitor_SMD:C_1206_3216Metric, B.Cu at (107.8, 118.8)
- added C10: CP, Capacitor_THT:CP_Radial_D5.0mm_P2.50mm, F.Cu at (91.2, 71.8)
- added C11: CP, Capacitor_THT:CP_Radial_D10.0mm_P5.00mm, F.Cu at (74.0, 71.0)
- added C12: CP, Capacitor_THT:CP_Radial_D10.0mm_P5.00mm, F.Cu at (107.6, 61.0)
- added C13: 0.1, Capacitor_SMD:C_1206_3216Metric, B.Cu at (86.1, 70.0)
- added C14: 0.1, Capacitor_SMD:C_1206_3216Metric, B.Cu at (85.2, 100.5)
- added C2: 0.1, Capacitor_SMD:C_1206_3216Metric, B.Cu at (88.6, 108.0)
- added C3: 0.1, Capacitor_SMD:C_1206_3216Metric, B.Cu at (88.6, 116.5)
- added C4: 0.1, Capacitor_SMD:C_1206_3216Metric, B.Cu at (92.5, 119.0)
- added C5: 0.1, Capacitor_SMD:C_1206_3216Metric, B.Cu at (93.8, 78.0)
- added C6: 0.1, Capacitor_SMD:C_1206_3216Metric, B.Cu at (91.2, 67.8)
- added C7: 0.1, Capacitor_SMD:C_1206_3216Metric, B.Cu at (91.2, 78.0)
- added C8: 0.1, Capacitor_SMD:C_1206_3216Metric, B.Cu at (81.2, 104.0)
- added C9: 0.1, Capacitor_SMD:C_1206_3216Metric, B.Cu at (88.8, 78.0)
- added D1: D, Diode_SMD:D_MELF, B.Cu at (98.0, 68.0)
- added D2: D, Diode_THT:D_DO-27_P15.24mm_Horizontal, F.Cu at (120.0, 55.0)
- added J1: POWER, Connector_Phoenix_MSTB:PhoenixContact_MSTBA_2,5_4-G-5,08_1x04_P5.08mm_Horizontal, F.Cu at (98.0, 61.0)
- added J2: UART, Connector_PinHeader_2.54mm:PinHeader_1x03_P2.54mm_Vertical, F.Cu at (121.7, 118.3)
- added R1: 1R0, Resistor_THT:R_Axial_DIN0207_L6.3mm_D2.5mm_P10.16mm_Horizontal, F.Cu at (83.2, 76.2)
- added R10: 4,7k, Resistor_SMD:R_0805_2012Metric, B.Cu at (110.3, 119.3)
- added R11: 4,7k, Resistor_SMD:R_0805_2012Metric, B.Cu at (95.0, 119.2)
- added R2: 10k, Resistor_SMD:R_0805_2012Metric, B.Cu at (85.6, 106.7)
- added R3: 10k, Resistor_SMD:R_0805_2012Metric, B.Cu at (85.6, 115.2)
- added R4: 10k, Resistor_SMD:R_0805_2012Metric, B.Cu at (85.8, 85.2)
- added R5: 10k, Resistor_SMD:R_0805_2012Metric, B.Cu at (85.7, 91.9)
- added R6: 10k, Resistor_SMD:R_0805_2012Metric, B.Cu at (85.8, 88.5)
- added R7: 1R0, Resistor_THT:R_Axial_DIN0207_L6.3mm_D2.5mm_P10.16mm_Horizontal, F.Cu at (86.1, 76.2)
- added R8: 47R, Resistor_SMD:R_0805_2012Metric, B.Cu at (112.8, 119.3)
- added R9: 47R, Resistor_SMD:R_0805_2012Metric, B.Cu at (97.5, 119.2)
- added REF**: SolderWirePad_1x01_Drill0.8mm, Connector_Wire:SolderWirePad_1x01_Drill0.8mm, F.Cu at (80.0, 76.3)
- added REF**: SolderWirePad_1x01_Drill0.8mm, Connector_Wire:SolderWirePad_1x01_Drill0.8mm, F.Cu at (78.0, 101.0)
- added REF**: SolderWirePad_1x01_Drill0.8mm, Connector_Wire:SolderWirePad_1x01_Drill0.8mm, F.Cu at (80.0, 81.9)
- added REF**: SolderWirePad_1x01_Drill0.8mm, Connector_Wire:SolderWirePad_1x01_Drill0.8mm, F.Cu at (87.0, 121.0)
- added REF**: SolderWirePad_1x01_Drill0.8mm, Connector_Wire:SolderWirePad_1x01_Drill0.8mm, F.Cu at (87.0, 125.0)
- added REF**: SolderWirePad_1x01_Drill0.8mm, Connector_Wire:SolderWirePad_1x01_Drill0.8mm, F.Cu at (92.0, 101.0)
- added REF**: MountingHole_3.2mm_M3, MountingHole:MountingHole_3.2mm_M3, F.Cu at (75.0, 124.0)
- added REF**: MountingHole_3.2mm_M3, MountingHole:MountingHole_3.2mm_M3, F.Cu at (127.0, 124.0)
- added REF**: MountingHole_3.2mm_M3, MountingHole:MountingHole_3.2mm_M3, F.Cu at (127.0, 54.0)
- added REF**: MountingHole_3.2mm_M3, MountingHole:MountingHole_3.2mm_M3, F.Cu at (75.0, 54.0)
- added RV1: 5k, Potentiometer_THT:Potentiometer_Piher_PT-6-V_Vertical, F.Cu at (80.0, 111.5)
- added RV2: 5k, Potentiometer_THT:Potentiometer_Piher_PT-6-V_Vertical, F.Cu at (80.0, 120.3)
- added SW1: RESET, Button_Switch_THT:SW_PUSH_6mm_H5mm, F.Cu at (124.0, 68.0)
- added SW2: RESET, Button_Switch_THT:SW_PUSH_6mm_H5mm, F.Cu at (116.0, 68.0)
- M1: value unicon_v1 -> UniCon
- moved U3 66.6 mm to (93.7, 123.0)
- moved U1 66.4 mm to (109.0, 123.0)
- moved U2 34.9 mm to (83.0, 97.0), turned to 90 degrees
- moved M1 17.3 mm to (96.0, 115.0)
Connections:
- M1 pad 1: /12VDC -> /12V1
- M1 pad 11: Net-(M1-Pad11) -> /L298_IN1
- M1 pad 12: Net-(M1-Pad12) -> /L298_IN2
- M1 pad 13: Net-(M1-Pad13) -> /L298_ENA
- M1 pad 19: Net-(M1-Pad19) -> /AD1
- M1 pad 2: /5VDC -> +5V
- M1 pad 20: Net-(M1-Pad20) -> /AD2
- M1 pad 21: Net-(M1-Pad21) -> /ADC
- M1 pad 27: Net-(M1-Pad27) -> /3VDC
- M1 pad 29: Net-(M1-Pad29) -> /~RST
- M1 pad 30: Net-(M1-Pad30) -> /BOOT
- M1 pad 39: Net-(M1-Pad39) -> /UART_TX
- M1 pad 40: Net-(M1-Pad40) -> /UART_RX
- M1 pad 45: Net-(M1-Pad45) -> /DHT1
- M1 pad 46: Net-(M1-Pad46) -> /DHT2
- U1 pad 2: /DHT1 -> Net-(R10-Pad1)
- U2 pad 1: Net-(R1-Pad1) -> /ADC
- U2 pad 10: /IN1 -> /L298_IN2
- U2 pad 11: /ENA -> /L298_ENA
- U2 pad 12: /IN2 -> /L298_IN1
- U2 pad 13: /MOTA -> /MOTB
- U2 pad 14: /MOTB -> /MOTA
- U2 pad 15: Net-(R1-Pad1) -> /ADC
- U2 pad 5: /IN1 -> /L298_IN1
- U2 pad 6: /ENA -> /L298_ENA
- U2 pad 7: /IN2 -> /L298_IN2
- U2 pad 9: /5VDC -> +5V
- U3 pad 2: /DHT2 -> Net-(R11-Pad1)
Routing:
- net +5V: track 0.00 -> 132.9 mm, vias 0 -> 2
- net /GND1: track 0.00 -> 95.9 mm
- net /12VDC: track 0.00 -> 81.7 mm, vias 0 -> 2
- net /ADC: track 0.00 -> 58.9 mm, vias 0 -> 2
- net /MOTB: track 0.00 -> 50.3 mm, vias 0 -> 2
- net /MOTA: track 0.00 -> 43.0 mm, vias 0 -> 2
- net /BOOT: track 0.00 -> 37.8 mm
- net /L298_ENA: track 0.00 -> 35.7 mm, vias 0 -> 4
- net /L298_IN1: track 0.00 -> 32.9 mm
- net /~RST: track 0.00 -> 30.3 mm
- net /DHT1: track 0.00 -> 28.1 mm
- net /3VDC: track 0.00 -> 28.1 mm
- net /L298_IN2: track 0.00 -> 26.9 mm
- net /12V1: track 0.00 -> 25.4 mm
- net GND: track 0.00 -> 23.6 mm
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- added copper zone on B.Cu, net GND
Other:
- board size 59 x 67 mm -> 60 x 78 mm
- net class power added: clearance 0.4, trace_width 0.6, via_dia 1.6, via_drill 0.7

Commit message: pcb ir schemos paruosimas
Parts:
- added D3: D, Diode_SMD:D_SMA, B.Cu at (83.5, 52.5)
- added D4: D, Diode_SMD:D_SMA, B.Cu at (91.0, 52.5)
- added D5: D, Diode_SMD:D_SMA, B.Cu at (83.5, 56.5)
- added D6: D, Diode_SMD:D_SMA, B.Cu at (91.0, 56.5)
- added R12: 4,7k, Resistor_SMD:R_0805_2012Metric, B.Cu at (115.3, 119.3)
- added R13: 4,7k, Resistor_SMD:R_0805_2012Metric, B.Cu at (100.1, 119.2)
- added REF**: SolderWirePad_1x01_Drill0.8mm, Connector_Wire:SolderWirePad_1x01_Drill0.8mm, F.Cu at (97.8, 130.5)
- added REF**: SolderWirePad_1x01_Drill0.8mm, Connector_Wire:SolderWirePad_1x01_Drill0.8mm, F.Cu at (97.8, 138.8)
- C5, C6: footprint Capacitor_SMD:C_1206_3216Metric -> Capacitor_SMD:C_0805_2012Metric
- C7, C9: value 0.1 -> 1.0
- moved C7 18.4 mm to (104.2, 65.0)
- moved C6 4.95 mm to (94.8, 71.2), turned to 270 degrees
- moved C9 4.93 mm to (91.2, 73.8)
- moved C5 3.16 mm to (94.8, 75.0), turned to 90 degrees
- moved C8 2.46 mm to (83.7, 104.2)
- moved REF** 2.00 mm to (80.0, 101.0)
- moved C10 1.50 mm to (91.2, 70.2), turned to 90 degrees
- moved C12 1.00 mm to (107.6, 62.0)
- moved RV2 0.05 mm to (80.0, 120.3)
Connections:
- C7 pad 1: /12V1 -> /12VDC
- C7 pad 2: GND -> /GND1
Routing:
- net /12VDC: track 81.7 -> 98.5 mm
- net /~RST: track 30.3 -> 46.1 mm
- net /MOTA: track 43.0 -> 56.6 mm
- net /BOOT: track 37.8 -> 50.8 mm
- net /MOTB: track 50.3 -> 58.8 mm
- net /12V1: track 25.4 -> 18.1 mm
- net +5V: track 132.9 -> 126.3 mm
- net /GND1: track 95.9 -> 101.3 mm
- net /DHT2: track 17.5 -> 20.0 mm
- net GND: track 23.6 -> 21.6 mm
Other:
- board size 60 x 78 mm -> 60 x 90 mm
- board text added: "RX"
- board text added: "TX"

Commit message: 2019-04-16
Routing:
- net /GND1: track 101.3 -> 49.6 mm
- net Net-(D1-Pad2): track 15.9 -> 16.7 mm
Changed lines of the file:
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@@
-(kicad_pcb (version 20171130) (host pcbnew "(5.1.0)-1")
+(kicad_pcb (version 20171130) (host pcbnew "(5.0.0)")
   (general
     (thickness 1.6)
     (drawings 15)
-    (tracks 291)
+    (tracks 284)
     (zones 0)
     (modules 55)
@@
   )
   (setup
-    (last_trace_width 0.6)
+    (last_trace_width 1)
     (user_trace_width 0.4)
     (user_trace_width 0.6)
@@
     (zone_45_only no)
     (trace_min 0.2)
+    (segment_width 0.2)
+    (edge_width 0.05)
     (via_size 0.8)
     (via_drill 0.4)
@@
     (uvia_min_size 0.2)
     (uvia_min_drill 0.1)
-    (edge_width 0.05)
-    (segment_width 0.2)
     (pcb_text_width 0.3)
     (pcb_text_size 1.5 1.5)
@@
     (mod_text_width 0.15)
     (pad_size 1.8 1.8)
-    (pad_drill 0.8)
+    (pad_drill 0.7)
     (pad_to_mask_clearance 0.051)
     (solder_mask_min_width 0.25)
@@
     (fp_arc (start 2.5 -2.5) (end 5.592 -3.564) (angle -98) (layer F.SilkS) (width 0.12))
     (fp_arc (start 2.5 -2.5) (end 2.5 0.77) (angle -71) (layer F.SilkS) (width 0.12))
-    (pad 1 thru_hole circle (at 0 0) (size 1.62 1.62) (drill 0.9) (layers *.Cu *.Mask)
+    (pad 1 thru_hole circle (at 0 0) (size 1.8 1.8) (drill 0.7) (layers *.Cu *.Mask)
       (net 1 +5V))
-    (pad 2 thru_hole circle (at 5 -2.5) (size 1.62 1.62) (drill 0.9) (layers *.Cu *.Mask)
+    (pad 2 thru_hole circle (at 5 -2.5) (size 1.8 1.8) (drill 0.7) (layers *.Cu *.Mask)
       (net 39 "Net-(R2-Pad2)"))
-    (pad 3 thru_hole circle (at 0 -5) (size 1.62 1.62) (drill 0.9) (layers *.Cu *.Mask)
+    (pad 3 thru_hole circle (at 0 -5) (size 1.8 1.8) (drill 0.7) (layers *.Cu *.Mask)
       (net 3 GND))
     (model ${KISYS3DMOD}/Potentiometer_THT.3dshapes/Potentiometer_Piher_PT-6-V_Vertical.wrl
@@
       (effects (font (size 1 1) (thickness 0.15)))
     )
-    (pad 3 thru_hole circle (at 0 -5) (size 1.62 1.62) (drill 0.9) (layers *.Cu *.Mask)
+    (pad 3 thru_hole circle (at 0 -5) (size 1.8 1.8) (drill 0.7) (layers *.Cu *.Mask)
       (net 3 GND))
-    (pad 2 thru_hole circle (at 5 -2.5) (size 1.62 1.62) (drill 0.9) (layers *.Cu *.Mask)
+    (pad 2 thru_hole circle (at 5 -2.5) (size 1.8 1.8) (drill 0.7) (layers *.Cu *.Mask)
       (net 40 "Net-(R3-Pad2)"))
-    (pad 1 thru_hole circle (at 0 0) (size 1.62 1.62) (drill 0.9) (layers *.Cu *.Mask)
+    (pad 1 thru_hole circle (at 0 0) (size 1.8 1.8) (drill 0.7) (layers *.Cu *.Mask)
       (net 1 +5V))
     (model ${KISYS3DMOD}/Potentiometer_THT.3dshapes/Potentiometer_Piher_PT-6-V_Vertical.wrl
@@
   (segment (start 83.04 94.5) (end 83 94.46) (width 0.8) (layer B.Cu) (net 33))
   (segment (start 86.4 94.5) (end 83.04 94.5) (width 0.8) (layer B.Cu) (net 33))
-  (segment (start 87.84 62.46) (end 87.84 61) (width 0.8) (layer B.Cu) (net 33))
-  (segment (start 82.46 81.76) (end 77.2 76.5) (width 0.8) (layer B.Cu) (net 33))
-  (segment (start 83 81.76) (end 82.46 81.76) (width 0.8) (layer B.Cu) (net 33))
-  (segment (start 77.2 76.5) (end 77.2 68.2) (width 0.8) (layer B.Cu) (net 33))
-  (segment (start 77.2 68.2) (end 81.4 64) (width 0.8) (layer B.Cu) (net 33))
-  (segment (start 81.4 64) (end 86.3 64) (width 0.8) (layer B.Cu) (net 33))
-  (segment (start 86.3 64) (end 87.84 62.46) (width 0.8) (layer B.Cu) (net 33))
   (segment (start 85.5 56.5) (end 89 56.5) (width 0.8) (layer B.Cu) (net 33))
   (segment (start 89 57.5) (end 89 56.5) (width 0.8) (layer B.Cu) (net 33))
   (segment (start 87.84 61) (end 87.84 58.66) (width 0.8) (layer B.Cu) (net 33))
   (segment (start 87.84 58.66) (end 89 57.5) (width 0.8) (layer B.Cu) (net 33))
+  (segment (start 87.84 63.16) (end 87.84 61) (width 0.8) (layer B.Cu) (net 33))
+  (segment (start 83 81.76) (end 82.46 81.76) (width 0.8) (layer B.Cu) (net 33))
+  (segment (start 77.2 76.5) (end 77.2 68.2) (width 0.8) (layer B.Cu) (net 33))
+  (segment (start 82.46 81.76) (end 77.2 76.5) (width 0.8) (layer B.Cu) (net 33))
+  (segment (start 77.2 68.2) (end 81.4 64) (width 0.8) (layer B.Cu) (net 33))
+  (segment (start 81.4 64) (end 87 64) (width 0.8) (layer B.Cu) (net 33))
+  (segment (start 87 64) (end 87.84 63.16) (width 0.8) (layer B.Cu) (net 33))
   (segment (start 125.34 112.46) (end 125.34 111.5) (width 0.4) (layer B.Cu) (net 34))
   (segment (start 124.6 113.2) (end 125.34 112.46) (width 0.4) (layer B.Cu) (net 34))
@@
   (segment (start 91.25 72.5) (end 92.5 72.5) (width 0.4) (layer B.Cu) (net 37))
   (segment (start 98 61) (end 98 65.6) (width 0.6) (layer B.Cu) (net 38))
-  (segment (start 104.76 58.49) (end 104.76 55) (width 1) (layer B.Cu) (net 38))
-  (segment (start 98 61) (end 102.25 61) (width 1) (layer B.Cu) (net 38))
-  (segment (start 102.25 61) (end 104.76 58.49) (width 1) (layer B.Cu) (net 38))
+  (segment (start 104.76 59.94) (end 104.76 55) (width 1) (layer B.Cu) (net 38))
+  (segment (start 98 61) (end 103.7 61) (width 1) (layer B.Cu) (net 38))
+  (segment (start 103.7 61) (end 104.76 59.94) (width 1) (layer B.Cu) (net 38))
   (segment (start 84.6625 106.7) (end 84.6625 107.6625) (width 0.4) (layer B.Cu) (net 39))
   (segment (start 85.045001 108.045001) (end 85.045001 109.025001) (width 0.4) (layer B.Cu) (net 39))
@@
   (segment (start 92.92 61) (end 92.92 56.58) (width 1) (layer B.Cu) (net 42))
   (segment (start 107.7 66.9) (end 107.6 67) (width 1) (layer B.Cu) (net 42))
-  (segment (start 112.75 57.25) (end 117.5 57.25) (width 1) (layer B.Cu) (net 42))
-  (segment (start 110.5 59.5) (end 112.75 57.25) (width 1) (layer B.Cu) (net 42))
-  (segment (start 110.5 65.75) (end 110.5 59.5) (width 1) (layer B.Cu) (net 42))
-  (segment (start 107.6 67) (end 109.25 67) (width 1) (layer B.Cu) (net 42))
-  (segment (start 109.25 67) (end 110.5 65.75) (width 1) (layer B.Cu) (net 42))
-  (segment (start 121.75 57.25) (end 117.35 57.25) (width 1) (layer B.Cu) (net 42))
   (segment (start 93 52.6) (end 93.1 52.5) (width 1) (layer B.Cu) (net 42))
   (segment (start 93 56.5) (end 93 52.6) (width 1) (layer B.Cu) (net 42))
-  (segment (start 93.1 52.5) (end 121.75 52.5) (width 1) (layer B.Cu) (net 42))
-  (segment (start 121.75 52.5) (end 122.75 53.5) (width 1) (layer B.Cu) (net 42))
-  (segment (start 122.75 53.5) (end 122.75 56.25) (width 1) (layer B.Cu) (net 42))
-  (segment (start 122.75 56.25) (end 121.75 57.25) (width 1) (layer B.Cu) (net 42))
   (segment (start 104.25 66.4) (end 104.25 67) (width 1) (layer B.Cu) (net 42))
   (segment (start 88.61 66.09) (end 83.01 66.09) (width 1) (layer B.Cu) (net 42))
@@
   (segment (start 101.1 67.5) (end 95.6 67.5) (width 1) (layer B.Cu) (net 42))
   (segment (start 95.6 67.5) (end 93.6 65.5) (width 1) (layer B.Cu) (net 42))
-  (segment (start 93.6 65.5) (end 89.2 65.5) (width 1) (layer B.Cu) (net 42))
   (segment (start 89.2 65.5) (end 88.61 66.09) (width 1) (layer B.Cu) (net 42))
+  (segment (start 92.92 65.42) (end 93 65.5) (width 1) (layer B.Cu) (net 42))
+  (segment (start 92.92 61) (end 92.92 65.42) (width 1) (layer B.Cu) (net 42))
+  (segment (start 93.6 65.5) (end 93 65.5) (width 1) (layer B.Cu) (net 42))
+  (segment (start 93 65.5) (end 89.2 65.5) (width 1) (layer B.Cu) (net 42))
   (segment (start 85.7375 84.3) (end 85.75 84.3125) (width 0.4) (layer B.Cu) (net 43))
   (segment (start 83 84.3) (end 85.7375 84.3) (width 0.4) (layer B.Cu) (net 43))

Commit message: 2019-04-17
Parts:
- added REF**: SolderWirePad_1x01_Drill0.8mm, Connector_Wire:SolderWirePad_1x01_Drill0.8mm, F.Cu at (126.2, 130.2)
- added REF**: SolderWirePad_1x01_Drill0.8mm, Connector_Wire:SolderWirePad_1x01_Drill0.8mm, F.Cu at (126.8, 138.8)
Other:
- outline, holes or cut-outs redrawn
